File: VTOL_Board/mcu.kicad_sch (KiCad schematic)
At the start: 21 parts, among them J201 ICSP, SW201 RESET, SW202 START_SW, SW203 STOP/MODE_SW, U201 ATmega328P, Y201 16mHz

Commit message: Modify boilerplate for vtol
Other:
- title: Inverted Pendulum Controller -> VTOL Board
Changed lines of the file:
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@@
   (paper "A4")
   (title_block
-    (title "Inverted Pendulum Controller")
+    (title "VTOL Board")
     (date "${ISSUE}")
     (rev "${REVISION}")
