File: VTOL_Board/prog.kicad_sch (KiCad schematic)
At the start: 14 parts, among them J401 USB_B_Micro, J402 PROG, U401 FT232RL

Commit message: Modify boilerplate for vtol
Other:
- title: Inverted Pendulum Controller -> VTOL Board
Changed lines of the file:
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@@
   (paper "A4")
   (title_block
-    (title "Inverted Pendulum Controller")
+    (title "VTOL Board")
     (date "${ISSUE}")
     (rev "${REVISION}")
